File: limiter-distortion.kicad_pcb (KiCad board)
At the start: 2 copper layers, 62 x 60 mm, 59 parts, among them J1 Input, J2 10K Pot, J3 PS, J4 Pot 10k x2, J5 SW distortion, J6 SW limiter, J7 Output, J8 Input, Q1 J309, Q2 MMBT3904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

Commit message: 1
Parts:
- added J9: pedal distortion, Connector_PinHeader_2.54mm:PinHeader_1x02_P2.54mm_Vertical, F.Cu at (114.5, 132.0)
- R8, R9: value 150 -> 330
Routing:
- net Net-(J5-Pin_1): track 29.3 -> 38.2 mm
- net Net-(D3-A): track 48.4 -> 53.4 mm
- net Net-(U1C-V+): track 17.4 -> 15.8 mm
