File: limiter-distortion.kicad_sch (KiCad schematic)
At the start: 59 parts, among them J1 Input, J2 10K Pot, J3 PS, J4 Pot 10k x2, J5 SW distortion, J6 SW limiter, J7 Output, J8 Input, Q1 J309, Q2 MMBT3904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

Commit message: 1
Parts:
- added J9: pedal distortion, Connector_PinHeader_2.54mm:PinHeader_1x02_P2.54mm_Vertical, symbol Connector:Conn_01x02_Socket
- R8, R9: value 150 -> 330
Connections:
- net at J5.1 (Pin_1), J6.2 (Pin_2), U2.3 (+): now also J9.1 (Pin_1)
- net at D3.2 (A), D4.1 (K), J4.1 (Pin_1)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: now also J9.2 (Pin_2)
Changed lines of the file:
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@@
 	)
 	(junction
+		(at 205.74 63.5)
+		(diameter 0)
+		(color 0 0 0 0)
+	)
+	(junction
 		(at 127 99.06)
 		(diameter 0)
@@
 	(wire
 		(pts
+			(xy 205.74 63.5) (xy 205.74 67.31)
+		)
+		(stroke
+			(width 0)
+			(type default)
+		)
+	)
+	(wire
+		(pts
 			(xy 233.68 76.2) (xy 243.84 76.2)
 		)
@@
 	(wire
 		(pts
+			(xy 233.68 63.5) (xy 205.74 63.5)
+		)
+		(stroke
+			(width 0)
+			(type default)
+		)
+	)
+	(wire
+		(pts
 			(xy 218.44 92.71) (xy 218.44 102.87)
 		)
@@
 	(wire
 		(pts
-			(xy 205.74 39.37) (xy 205.74 67.31)
+			(xy 205.74 39.37) (xy 205.74 63.5)
 		)
 		(stroke
@@
 	(wire
 		(pts
+			(xy 233.68 67.31) (xy 233.68 63.5)
+		)
+		(stroke
+			(width 0)
+			(type default)
+		)
+	)
+	(wire
+		(pts
 			(xy 73.66 33.02) (xy 73.66 36.83)
 		)
@@
 	(wire
 		(pts
+			(xy 233.68 69.85) (xy 233.68 76.2)
+		)
+		(stroke
+			(width 0)
+			(type default)
+		)
+	)
+	(wire
+		(pts
 			(xy 161.29 116.84) (xy 161.29 118.11)
 		)
@@
 	(label "+1V"
 		(at 82.55 120.65 0)
+		(fields_autoplaced yes)
 		(effects
 			(font
@@
 	(label "-22V"
 		(at 33.02 50.8 0)
+		(fields_autoplaced yes)
 		(effects
 			(font
@@
 	(label "+22V"
 		(at 33.02 24.13 0)
+		(fields_autoplaced yes)
 		(effects
 			(font
@@
 	(label "Input"
 		(at 200.66 54.61 180)
+		(fields_autoplaced yes)
 		(effects
 			(font
@@
 	(label "MOD"
 		(at 106.68 123.19 0)
+		(fields_autoplaced yes)
 		(effects
 			(font
@@
 	(label "Input"
 		(at 43.18 68.58 0)
+		(fields_autoplaced yes)
 		(effects
 			(font
@@
 			)
 		)
-		(property "Value" "150"
+		(property "Value" "330"
 			(at 40.64 48.26 90)
 			(effects
@@
 			)
 		)
-		(property "Value" "150"
+		(property "Value" "330"
 			(at 40.64 21.59 90)
 			(effects
@@
 					(unit 1)
 				)
+			)
+		)
+	)
+	(symbol
+		(lib_id "Connector:Conn_01x02_Socket")
+		(at 238.76 67.31 0)
+		(unit 1)
+		(exclude_from_sim no)
+		(in_bom yes)
+		(on_board yes)
+		(dnp no)
+		(fields_autoplaced yes)
+		(property "Reference" "J9"
+			(at 240.03 67.3099 0)
+			(effects
+				(font
+					(size 1.27 1.27)
+				)
+				(justify left)
+			)
+		)
+		(property "Value" "pedal distortion"
+			(at 240.03 69.8499 0)
+			(effects
+				(font
+					(size 1.27 1.27)
+				)
+				(justify left)
+			)
+		)
+		(property "Footprint" "Connector_PinHeader_2.54mm:PinHeader_1x02_P2.54mm_Vertical"
+			(at 238.76 67.31 0)
+			(effects
+				(font
+					(size 1.27 1.27)
+				)
+				(hide yes)
+			)
+		)
+		(property "Datasheet" "~"
+			(at 238.76 67.31 0)
+			(effects
+				(font
+					(size 1.27 1.27)
+				)
+				(hide yes)
+			)
+		)
+		(property "Description" "Generic connector, single row, 01x02, script generated"
+			(at 238.76 67.31 0)
+			(effects
+				(font
+					(size 1.27 1.27)
+				)
+				(hide yes)
+			)
+		)
+		(pin "2"
+		)
+		(pin "1"
+		)
+		(instances
+			(project "limiter-distortion"
+				(path "/ed4ae933-69cf-42d6-a171-9a67c59f030e"
+					(reference "J9")
+					(unit 1)
+				)
